File: Eagle/untitled.brd (EAGLE design)
At the start: 25.4 x 48.1 mm, 26 parts, among them T1 IRLML2502, T2 IRLML2502, T4 IRLML2502

Commit message: Rename Relays
Connections:
- net IN renamed INPUT
- net NR renamed OPEN
- net SW1 renamed RELAY1
- net SW2 renamed RELAY2
Changed lines of the file:
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@@
 <wire x1="5.334" y1="31.158" x2="5.25" y2="31.242" width="0.4064" layer="16"/>
 </signal>
-<signal name="IN">
+<signal name="INPUT">
 <contactref element="U$8" pad="5"/>
 <contactref element="R18" pad="2"/>
@@
 <wire x1="20" y1="29.21" x2="20.066" y2="29.276" width="0.4064" layer="16"/>
 </signal>
-<signal name="NR">
+<signal name="OPEN">
 <contactref element="R2" pad="1"/>
 <contactref element="J2" pad="13"/>
@@
 <wire x1="5.842" y1="22.098" x2="3.81" y2="24.13" width="0.4064" layer="1"/>
 </signal>
-<signal name="SW1">
+<signal name="RELAY1">
 <contactref element="R4" pad="1"/>
 <contactref element="J2" pad="5"/>
@@
 <wire x1="22.606" y1="18.034" x2="24.13" y2="16.51" width="0.4064" layer="16"/>
 </signal>
-<signal name="SW2">
+<signal name="RELAY2">
 <contactref element="R6" pad="1"/>
 <contactref element="J2" pad="6"/>
