File: Eagle/untitled.sch (EAGLE design)
At the start: 26 parts, among them T1 IRLML2502, T2 IRLML2502, T4 IRLML2502

Commit message: Rename Relays
Connections:
- net IN renamed INPUT
- net NR renamed OPEN
- net SW1 renamed RELAY1
- net SW2 renamed RELAY2
Changed lines of the file:
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@@
 </segment>
 </net>
-<net name="IN" class="0">
+<net name="INPUT" class="0">
 <segment>
 <pinref part="U$8" gate="G$1" pin="COL"/>
@@
 </segment>
 </net>
-<net name="NR" class="0">
+<net name="OPEN" class="0">
 <segment>
 <pinref part="R2" gate="G$1" pin="1"/>
@@
 </segment>
 </net>
-<net name="SW1" class="0">
+<net name="RELAY1" class="0">
 <segment>
 <pinref part="R4" gate="G$1" pin="1"/>
@@
 </segment>
 </net>
-<net name="SW2" class="0">
+<net name="RELAY2" class="0">
 <segment>
 <pinref part="R6" gate="G$1" pin="1"/>
